File: Power Supply/Boards/12V10A supply.brd (EAGLE design)
At the start: 57 x 44 mm, 11 parts, among them U1 LMZ12010

Commit message: Updated Schematics and Board file Added BOM for Power Supply Added Data sheets for Power Supply
Parts:
- renumbered JP1 to J2, U$1 to J1, VOUTJACK to J3
Changed lines of the file:
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@@
 <attribute name="MFG_PN" value="APXA160ARA331MJC0G" x="44" y="24.75" size="1.778" layer="27" rot="R270" display="off"/>
 </element>
-<element name="VOUTJACK" library="Texas Instruments" package="2PINTERMINAL" value="MC24356" x="51.95" y="4.2" rot="R90"/>
-<element name="JP1" library="SparkFun-Connectors" package="1X02" value="" x="51.05" y="14"/>
-<element name="U$1" library="Texas Instruments" package="0050362375" value="5569-02A2MS-225" x="2.8" y="13.95"/>
+<element name="J3" library="Texas Instruments" package="2PINTERMINAL" value="MC24356" x="51.95" y="4.2" rot="R90"/>
+<element name="J2" library="SparkFun-Connectors" package="1X02" value="" x="51.05" y="14"/>
+<element name="J1" library="Texas Instruments" package="0050362375" value="5569-02A2MS-225" x="2.8" y="13.95"/>
 </elements>
 <signals>
@@
 <contactref element="CIN2" pad="2"/>
 <contactref element="CIN3" pad="2"/>
-<contactref element="VOUTJACK" pad="-"/>
+<contactref element="J3" pad="-"/>
 <via x="25.75" y="37.715" extent="1-16" drill="0.3302"/>
 <via x="27.25" y="37.715" extent="1-16" drill="0.3302"/>
@@
 <via x="37.875" y="41.215" extent="1-16" drill="0.3302"/>
 <via x="37.875" y="39.715" extent="1-16" drill="0.3302"/>
-<contactref element="JP1" pad="2"/>
+<contactref element="J2" pad="2"/>
 <via x="37.875" y="28.715" extent="1-16" drill="0.3302"/>
 <via x="37.875" y="27.215" extent="1-16" drill="0.3302"/>
-<contactref element="U$1" pad="2"/>
+<contactref element="J1" pad="2"/>
 <via x="24.25" y="1.715" extent="1-16" drill="0.3302"/>
 <via x="26.25" y="1.715" extent="1-16" drill="0.3302"/>
@@
 <vertex x="5.125" y="0"/>
 </polygon>
-<contactref element="U$1" pad="1"/>
+<contactref element="J1" pad="1"/>
 <wire x1="2.8" y1="13.95" x2="8.05" y2="13.95" width="2.54" layer="1"/>
 <wire x1="8.05" y1="13.95" x2="9" y2="13" width="0.8128" layer="1"/>
@@
 <contactref element="RFBT" pad="2"/>
 <contactref element="CO1" pad="+"/>
-<contactref element="VOUTJACK" pad="+"/>
+<contactref element="J3" pad="+"/>
 <polygon width="0.3048" layer="1">
 <vertex x="32.74" y="23.3"/>
@@
 <vertex x="52" y="23.3"/>
 </polygon>
-<contactref element="JP1" pad="1"/>
+<contactref element="J2" pad="1"/>
 </signal>
 <signal name="N$4">
