File: Power Supply/Boards/12V10A supply.sch (EAGLE design)
At the start: 11 parts, among them U1 LMZ12010

Commit message: Updated Schematics and Board file Added BOM for Power Supply Added Data sheets for Power Supply
Parts:
- renumbered JP1 to J2, U$1 to J1, VOUTJACK to J3
Changed lines of the file:
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@@
 <part name="GND7" library="SparkFun-Aesthetics" deviceset="GND" device=""/>
 <part name="GND8" library="SparkFun-Aesthetics" deviceset="GND" device=""/>
-<part name="VOUTJACK" library="Texas Instruments" deviceset="MC24356" device=""/>
+<part name="J3" library="Texas Instruments" deviceset="MC24356" device=""/>
 <part name="GND2" library="SparkFun-Aesthetics" deviceset="GND" device=""/>
-<part name="JP1" library="SparkFun-Connectors" deviceset="M02" device="PTH"/>
+<part name="J2" library="SparkFun-Connectors" deviceset="M02" device="PTH"/>
 <part name="GND10" library="SparkFun-Aesthetics" deviceset="GND" device=""/>
-<part name="U$1" library="Texas Instruments" deviceset="5569" device="-02A2MS-225"/>
+<part name="J1" library="Texas Instruments" deviceset="5569" device="-02A2MS-225"/>
 <part name="GND11" library="SparkFun-Aesthetics" deviceset="GND" device=""/>
 </parts>
@@
 <instance part="GND7" gate="1" x="35.56" y="22.86"/>
 <instance part="GND8" gate="1" x="27.94" y="22.86"/>
-<instance part="VOUTJACK" gate="G$1" x="142.24" y="48.26"/>
+<instance part="J3" gate="G$1" x="142.24" y="48.26"/>
 <instance part="GND2" gate="1" x="129.54" y="35.56"/>
-<instance part="JP1" gate="G$1" x="137.16" y="73.66" rot="R180"/>
+<instance part="J2" gate="G$1" x="137.16" y="73.66" rot="R180"/>
 <instance part="GND10" gate="1" x="129.54" y="66.04"/>
-<instance part="U$1" gate="G$1" x="2.54" y="48.26" rot="MR0"/>
+<instance part="J1" gate="G$1" x="2.54" y="48.26" rot="MR0"/>
 <instance part="GND11" gate="1" x="15.24" y="38.1"/>
 </instances>
@@
 </segment>
 <segment>
-<pinref part="VOUTJACK" gate="G$1" pin="-"/>
+<pinref part="J3" gate="G$1" pin="-"/>
 <pinref part="GND2" gate="1" pin="GND"/>
 <wire x1="129.54" y1="43.18" x2="129.54" y2="38.1" width="0.1524" layer="91"/>
@@
 <segment>
 <pinref part="GND10" gate="1" pin="GND"/>
-<pinref part="JP1" gate="G$1" pin="2"/>
+<pinref part="J2" gate="G$1" pin="2"/>
 <wire x1="129.54" y1="68.58" x2="129.54" y2="71.12" width="0.1524" layer="91"/>
 </segment>
 <segment>
-<pinref part="U$1" gate="G$1" pin="-"/>
+<pinref part="J1" gate="G$1" pin="-"/>
 <pinref part="GND11" gate="1" pin="GND"/>
 <wire x1="15.24" y1="43.18" x2="15.24" y2="40.64" width="0.1524" layer="91"/>
@@
 <junction x="43.18" y="53.34"/>
 <junction x="27.94" y="53.34"/>
-<pinref part="U$1" gate="G$1" pin="+"/>
+<pinref part="J1" gate="G$1" pin="+"/>
 <wire x1="15.24" y1="53.34" x2="27.94" y2="53.34" width="0.1524" layer="91"/>
 </segment>
@@
 <pinref part="CO1" gate="G$1" pin="+"/>
 <junction x="106.68" y="53.34"/>
-<pinref part="VOUTJACK" gate="G$1" pin="+"/>
+<pinref part="J3" gate="G$1" pin="+"/>
 <wire x1="129.54" y1="53.34" x2="116.84" y2="53.34" width="0.1524" layer="91"/>
 <junction x="116.84" y="53.34"/>
-<pinref part="JP1" gate="G$1" pin="1"/>
+<pinref part="J2" gate="G$1" pin="1"/>
 <wire x1="129.54" y1="73.66" x2="116.84" y2="73.66" width="0.1524" layer="91"/>
 <wire x1="116.84" y1="73.66" x2="116.84" y2="53.34" width="0.1524" layer="91"/>
